File: Hardware/Top/Set-Mile-TOP.sch (EAGLE design)
At the start: 19 parts, among them U2 NRF52832_MODULE_MDBT42

Commit message: Top Board Electronics Placed
Parts:
- removed SW4: (no value), LinnesLab-Switches:SPST-PTS830GG140-COPY.1-3
- added C13, C15, C17, C18, C19: 2.2uF, LinnesLab-Passives:CAPACITOR0402
- added C16: 10uF, LinnesLab-Passives:CAPACITOR0603
- added C2, C5, C6: 1u, LinnesLab-Passives:CAPACITOR0603
- added C20, C21: 4.7u, LinnesLab-Passives:CAPACITOR0603
- added CHRG2: MCP73831, LinnesLab-Power:MCP73831
- added D4, D5: (no value), LinnesLab-DiscreteSemi:SCHOTTKY-USC
- added J2: (no value), LinnesLab-Connectors:CONN_02
- added LDO2: MIC5504, LinnesLab-Power:MIC5504
- added R11: (no value), LinnesLab-Passives:RESISTOR0603
- added R12, R13, R14, R15: 100k, LinnesLab-Passives:RESISTOR0603
- added R6, R8, R9: 10k, LinnesLab-Passives:RESISTOR0603
- added R7: 390k, LinnesLab-Passives:RESISTOR0603
- added SD2: (no value), LinnesLab-Connectors:MICROSD
- added SW1: (no value), LinnesLab-Switches:SPST-PTS830GG140-COPY.1-3
- added U$1, U$2, U$3: SWITCH.MOM, LinnesLab-Switches:SWITCH.MOM
- added U3: (no value), LinnesLab-Displays:DISP_OLED_UG-2864HSWEG01-NO-WRAPAROUND
- added U4: PCF8523, LinnesLab-Clocks:PCF8523
- added USB2: USB.MICRO-BIGGERPADS, LinnesLab-Connectors:USB.MICRO-BIGGERPADS
- added XTAL3: 32.7680kHz, LinnesLab-Clocks:CRYSTALECS-.327-12.5-12-C-TR
Connections:
- new net BATT: R13.1, R14.2
- new net CD1: SD2.CARD_DETECT
- new net CD2: SD2.CARD_DETECT1
- new net CHRG.STAT: CHRG2.STAT, R12.1
- new net CS.OLED: U3./CS
- new net DC.OLED: U3.DC/I2C_SA0
- new net N$1: R6.2, U3.BS1
- new net N$13: C16.2, U3.VCC
- new net N$15: C18.2, U3.VCOMH
- new net N$17: CHRG2.PROG, R11.2
- new net N$19: U4.OSCO, XTAL3.1
- new net N$2: R7.1, U3.IREF
- new net N$20: U4.OSCI, XTAL3.2
- new net N$3: C13.2, U3.C2P
- new net N$5: C13.1, U3.C2N
- new net N$7: C15.2, U3.C1P
- new net N$8: C15.1, U3.C1N
- new net RESET.OLED: U3./RES
- new net SD.CS: SD2.CS
- new net SW1: U$1.1, U$2.1, U$3.1
- new net USB+: USB2.D+
- new net USB-: USB2.D-
- new net VBATT: U4.VBAT
- new net VIN: C21.2, C5.2, CHRG2.VIN, D4.C, D5.C, LDO2.EN, LDO2.IN, R12.2
- new net VLIPO: C20.1, CHRG2.VBAT, D4.A, J2.2, R13.2
- new net V_USB: D5.A, USB2.V+
- net 3.3V: now also C17.2, C19.2, C2.1, C6.1, LDO2.OUT, R15.2, R8.2, R9.2, SD2.VDD, U3.VBAT, U3.VDD, U4.VDD
- net DFU: now also SW1.B
- net GND: now also C16.1, C17.1, C18.1, C19.1, C2.2, C20.2, C21.1, C5.1, C6.2, CHRG2.VSS, J2.1, LDO2.GND, R11.1, R14.1, R15.1, R6.1, R7.2, SD2.GND, SD2.GND1, SD2.VSS, SW1.A, U$1.3, U$1.4, U$2.3, U$2.4, U$3.3, U$3.4, U3.BS0, U3.BS2, U3.NC(GND)@1, U3.NC(GND)@2, U3.VLSS, U3.VSS, U4.VSS, USB2.GND, USB2.SHIELD; no longer SW4.B
- net MISO: now also SD2.DATA_OUT
- net MOSI: now also SD2.DATA_IN, U3.D1/SPI_SDIN/I2C_SDA
- net RESET: no longer SW4.A
- net SCK: now also SD2.SCLK, U3.D0/SPI_SCLK/I2C_SCK
- net SCL: now also R8.1, U4.SCL
- net SDA: now also R9.1, U4.SDA
Other:
- note added: "Back-up battery if desired"
- note added: "Buttons"
- note added: "Connect MISO, MOSI, and SCK to appropriate pins on microcontroller. Those are SPI pins and are generally prespecified. You have more flexibility with the SD.CS pin."
- note added: "Cortex Debugger/ Programmer"
- note added: "Digital Outputs CS OLED RESET.OLED DC.OLED Digital Inputs 3x Buttons Charge Status Analog Inputs Battery Monitor Analog Outputs"
- note added: "I2C Address = 0x68h"
- note added: "OLED"
- note added: "Power Management"
- note added: "RTC"
- note added: "Real-Time Clock"
- note added: "SD Card"
- note added: "nRFS2832 Module"
- moved on the sheet: C10, C11, C12, C14, C7, C8, C9, CORTEX1, D1, L2, LED3, LED4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

Commit message: updated board design to section 2
Parts:
- removed U$3: SWITCH.MOM, LinnesLab-Switches:SWITCH.MOM
- added C22: 100n, LinnesLab-Passives:CAPACITOR0603
- added C23, C24: 47p, LinnesLab-Passives:CAPACITOR0603
- added J1: (no value), LinnesLab-Connectors:CONN_07
- added JP2: (no value), LinnesLab-Switches:JUMPER-SMT_2_NO_SILK
- added LED5: RED, LinnesLab-LED:LED0603
- added LED6: YELLOW, LinnesLab-LED:LED0603
- added R1, R2: 0, LinnesLab-Passives:RESISTOR0603
- added R17, R18: 27, LinnesLab-Passives:RESISTOR0603
- added R19, R20: 1k, LinnesLab-Passives:RESISTOR0603
- added U5: FT231XS, LinnesLab-DigitalIC:FT231XS
- renumbered U$1 to SWITCH1, U$2 to SWITCH2
Connections:
- removed net BATT: R13.1, R14.2
- removed net CD1: SD2.CARD_DETECT
- removed net CHRG.STAT: CHRG2.STAT, R12.1
- removed net CS.OLED: U3./CS
- removed net DC.OLED: U3.DC/I2C_SA0
- removed net RESET.OLED: U3./RES
- removed net RXD: U2.P0.08
- removed net SD.CS: SD2.CS
- removed net SW1: SWITCH1.1, SWITCH2.1, U$3.1
- removed net TXD: U2.P0.06
- removed net VBATT: U4.VBAT
- new net !CTS: JP2.2, U5.!CTS
- new net !DTR: U5.!DTR
- new net A4/BATT: R13.1, R14.2, U2.P0.28/AIN4
- new net A6/TIA: J1.5, U2.P0.30/AIN6
- new net A7/PPG: J1.7, U2.P0.31/AIN7
- new net D11/SW1: SWITCH1.1, U2.P0.11
- new net D15/SW2: SWITCH2.1, U2.P0.15
- new net D16/CS.OLED: U2.P0.16, U3./CS
- new net D27/CHRG.STATUS: CHRG2.STAT, R12.1, U2.P0.27
- new net D29/LED.CTRL: J1.6
- new net D3/RESET.OLED: U2.P0.03/AIN1, U3./RES
- new net D4/DC.OLED: U2.P0.02/AIN0, U2.P0.04/AIN2, U3.DC/I2C_SA0
- new net D5/CD1: SD2.CARD_DETECT, U2.P0.05/AIN3
- new net D7/SD.CS: SD2.CS, U2.P0.07
- new net D9/LED.CTRL: U2.P0.29/AIN5
- new net FT3V3: U5.3V3OUT
- new net N$23: R17.2, U5.USBDM
- new net N$24: R18.2, U5.USBDP
- new net N$25: LED5.C, R19.2
- new net N$26: LED6.C, R20.2
- new net RXD.FT: R2.1, U5.RXD
- new net RXD.NRF: R1.2, U2.P0.08
- new net RXLED: R19.1, U5.CBUS1
- new net TXD.FT: R1.1, U5.TXD
- new net TXD.NRF: R2.2, U2.P0.06
- new net TXLED: R20.1, U5.CBUS2
- net 3.3V: now also C22.2, LED5.A, LED6.A, U5.!RESET, U5.VCCIO
- net GND: now also C22.1, C23.2, C24.1, JP2.1, U5.GND@16, U5.GND@6; no longer U$3.3, U$3.4
- net SCL: now also R9.1; no longer R8.1
- net SDA: now also R8.1; no longer R9.1
- net USB+: now also C23.1, R18.1
- net USB-: now also C24.2, R17.1
- net V_USB: now also U5.VCC
Other:
- note added: "Digital Output"
- note added: "FTDI Serial-to-USB Converter"
- note added: "I don't remember if CTS needs to be grounded or left floating so here's a jumper to ground so it can be configued either way dynamically."
- note added: "TXD goes to RX on the other device RXD goes to TX on the other device"
- moved on the sheet: R8, R9

Commit message: routing bottom board and oranized top board
Parts:
- removed C22: 100n, LinnesLab-Passives:CAPACITOR0603
- removed C23, C24: 47p, LinnesLab-Passives:CAPACITOR0603
- removed C7: 1u, LinnesLab-Passives:CAPACITOR0603
- removed C8: (no value), LinnesLab-Passives:CAPACITOR0603
- removed CHRG2: MCP73831, LinnesLab-Power:MCP73831
- removed CORTEX1: CORTEX_DEBUG_PTH, LinnesLab-Connectors:CORTEX_DEBUG_PTH
- removed D4, D5: (no value), LinnesLab-DiscreteSemi:SCHOTTKY-USC
- removed JP2: (no value), LinnesLab-Switches:JUMPER-SMT_2_NO_SILK
- removed L2: 10u, LinnesLab-Passives:INDUCTOR0603
- removed LDO2: MIC5504, LinnesLab-Power:MIC5504
- removed LED5: RED, LinnesLab-LED:LED0603
- removed LED6: YELLOW, LinnesLab-LED:LED0603
- removed R19, R20: 1k, LinnesLab-Passives:RESISTOR0603
- removed SD2: (no value), LinnesLab-Connectors:MICROSD
- removed SWITCH1, SWITCH2: SWITCH.MOM, LinnesLab-Switches:SWITCH.MOM
- removed U4: PCF8523, LinnesLab-Clocks:PCF8523
- removed U5: FT231XS, LinnesLab-DigitalIC:FT231XS
- removed USB2: USB.MICRO-BIGGERPADS, LinnesLab-Connectors:USB.MICRO-BIGGERPADS
- removed XTAL3: 32.7680kHz, LinnesLab-Clocks:CRYSTALECS-.327-12.5-12-C-TR
- added C1: 1u, LinnesLab-Passives:CAPACITOR0603
- added C3: (no value), LinnesLab-Passives:CAPACITOR0603
- added C4: 4.7u, LinnesLab-Passives:CAPACITOR0603
- added CHRG1: MCP73831, LinnesLab-Power:MCP73831
- added D2, D3: (no value), LinnesLab-DiscreteSemi:SCHOTTKY-USC
- added DEBUG1: CORTEX_DEBUG_PTH, LinnesLab-Connectors:CORTEX_DEBUG_PTH
- added JP1: (no value), LinnesLab-Switches:JUMPER-SMT_2_NO_SILK
- added L1: 10u, LinnesLab-Passives:INDUCTOR0603
- added LDO1: MIC5504, LinnesLab-Power:MIC5504
- added LED1: RED, LinnesLab-LED:LED0603
- added LED2: BLUE, LinnesLab-LED:LED0603
- added R10: 10k, LinnesLab-Passives:RESISTOR0603
- added R16: 1k, LinnesLab-Passives:RESISTOR0603
- added RTC1: PCF8523, LinnesLab-Clocks:PCF8523
- added SD1: (no value), LinnesLab-Connectors:MICROSD
- added SW2: (no value), LinnesLab-Switches:SPST-PTS830GG140-COPY.1-3
- added SW4: SWITCH.MOM, LinnesLab-Switches:SWITCH.MOM
- added U1: NRF52832_MODULE_MDBT42, LinnesLab-Microcontrollers:NRF52832_MODULE_MDBT42
- added USB1: USB.MICRO-BIGGERPADS, LinnesLab-Connectors:USB.MICRO-BIGGERPADS
- added XTAL1: 32.768kHz, LinnesLab-Clocks:CRYSTALECS-.327-12.5-12-C-TR
- C10: value 300p -> 4.7u
- C11: value 300p -> 100n
- C12: value 10u -> 47p; device LinnesLab-Passives:CAPACITOR0805 -> LinnesLab-Passives:CAPACITOR0603
- C13: value 2.2uF -> 47p; device LinnesLab-Passives:CAPACITOR0402 -> LinnesLab-Passives:CAPACITOR0603
- C14: value 100n -> 10uF
- C15: value 2.2uF -> 100n; device LinnesLab-Passives:CAPACITOR0402 -> LinnesLab-Passives:CAPACITOR0603
- C16: value 10uF -> 2.2uF; device LinnesLab-Passives:CAPACITOR0603 -> LinnesLab-Passives:CAPACITOR0402
- C2: value 1u -> 10u; device LinnesLab-Passives:CAPACITOR0603 -> LinnesLab-Passives:CAPACITOR0805
- C20: value 4.7u -> 2.2uF; device LinnesLab-Passives:CAPACITOR0603 -> LinnesLab-Passives:CAPACITOR0402
- C21: value 4.7u -> 1u
- C5: value 1u -> (none)
- C9: value (none) -> 1u
- J1: device LinnesLab-Connectors:CONN_07 -> LinnesLab-Connectors:CONN_02
- J2: device LinnesLab-Connectors:CONN_02 -> LinnesLab-Connectors:CONN_07-1.27MM
- LED4: value BLUE -> YELLOW
- R1, R2: value 0 -> 10k
- R11: value (none) -> 10k
- R12, R13: value 100k -> 27
- R14: value 100k -> 390k
- R15: value 100k -> 1k
- R17, R18: value 27 -> 0
- R3: value 1k -> 100k
- R4: value 1k -> (none)
- R5: value 10k -> 1k
- R6, R8, R9: value 10k -> 100k
- R7: value 390k -> 1k
- SW3: value (none) -> SWITCH.MOM; device LinnesLab-Switches:SPST-PTS830GG140-COPY.1-3 -> LinnesLab-Switches:SWITCH.MOM
- U2: value NRF52832_MODULE_MDBT42 -> FT231XS; device LinnesLab-Microcontrollers:NRF52832_MODULE_MDBT42 -> LinnesLab-DigitalIC:FT231XS
- XTAL2: value 32.768kHz -> 32.7680kHz
Connections:
- net !CTS: now also JP1.2, U2.!CTS; no longer JP2.2, U5.!CTS
- net !DTR: now also U2.!DTR; no longer U5.!DTR
- net 3.3V: now also C15.2, C2.2, C20.2, C21.1, C9.1, D3.C, DEBUG1.VCC, J2.4, LDO1.OUT, LED3.A, LED4.A, R1.2, R10.2, R2.2, R6.2, RTC1.VDD, SD1.VDD, U1.VDD, U2.!RESET, U2.VCCIO; no longer C12.2, C17.2, C2.1, C22.2, C6.1, CORTEX1.VCC, D1.C, LDO2.OUT, LED5.A, LED6.A, R15.2, R5.2, R8.2, R9.2, SD2.VDD, U2.VDD, U4.VDD, U5.!RESET, U5.VCCIO
- net A4/BATT: now also R8.1, R9.2, U1.P0.28/AIN4; no longer R13.1, R14.2, U2.P0.28/AIN4
- net A6/TIA: now also J2.6, U1.P0.30/AIN6; no longer J1.5, U2.P0.30/AIN6
- net A7/PPG: now also J2.7, U1.P0.31/AIN7; no longer J1.7, U2.P0.31/AIN7
- net CD2: now also SD1.CARD_DETECT1; no longer SD2.CARD_DETECT1
- net D11/SW1: now also SW3.1, U1.P0.11; no longer SWITCH1.1, U2.P0.11
- net D15/SW2: now also SW4.1, U1.P0.15; no longer SWITCH2.1, U2.P0.15
- net D16/CS.OLED: now also U1.P0.16; no longer U2.P0.16
- net D27/CHRG.STATUS: now also CHRG1.STAT, R3.1, U1.P0.27; no longer CHRG2.STAT, R12.1, U2.P0.27
- net D29/LED.CTRL: now also J2.5; no longer J1.6
- net D3/RESET.OLED: now also U1.P0.03/AIN1; no longer U2.P0.03/AIN1
- net D4/DC.OLED: now also U1.P0.02/AIN0, U1.P0.04/AIN2; no longer U2.P0.02/AIN0, U2.P0.04/AIN2
- net D5/CD1: now also SD1.CARD_DETECT, U1.P0.05/AIN3; no longer SD2.CARD_DETECT, U2.P0.05/AIN3
- net D7/SD.CS: now also SD1.CS, U1.P0.07; no longer SD2.CS, U2.P0.07
- net D9/LED.CTRL: now also U1.P0.29/AIN5; no longer U2.P0.29/AIN5
- net DFU: now also SW2.B, U1.P0.20; no longer SW3.B, U2.P0.20
- net DTR: now also C11.1; no longer C14.1
- net FRST: now also U1.P0.22; no longer U2.P0.22
- net FT3V3: now also U2.3V3OUT; no longer U5.3V3OUT
- net GND: now also C1.2, C13.2, C14.1, C15.1, C2.1, C20.1, C21.2, C3.1, C4.1, C5.2, C6.1, CHRG1.VSS, DEBUG1.GND@3, DEBUG1.GND@5, DEBUG1.GNDDTCT, DEBUG1.KEY, J1.1, J2.3, JP1.1, LDO1.GND, LED1.C, LED2.C, R14.2, R4.1, R9.1, RTC1.VSS, SD1.GND, SD1.GND1, SD1.VSS, SW2.A, SW3.3, SW3.4, SW4.3, SW4.4, U1.GND@1, U1.GND@2, U1.GND@3, U1.GND@4, U2.GND@16, U2.GND@6, USB1.GND, USB1.SHIELD; no longer C11.2, C16.1, C18.1, C2.2, C20.2, C21.1, C22.1, C23.2, C24.1, C5.1, C6.2, C7.2, C8.1, CHRG2.VSS, CORTEX1.GND@3, CORTEX1.GND@5, CORTEX1.GNDDTCT, CORTEX1.KEY, J2.1, JP2.1, LDO2.GND, LED3.C, LED4.C, R14.1, R15.1, R7.2, SD2.GND, SD2.GND1, SD2.VSS, SW3.A, SWITCH1.3, SWITCH1.4, SWITCH2.3, SWITCH2.4, U2.GND@1, U2.GND@2, U2.GND@3, U2.GND@4, U4.VSS, U5.GND@16, U5.GND@6, USB2.GND, USB2.SHIELD
- net LED1: now also R5.2, U1.P0.17; no longer R3.2, U2.P0.17
- net LED2: now also R7.2, U1.P0.19; no longer R4.2, U2.P0.19
- net MISO: now also SD1.DATA_OUT, U1.P0.14; no longer SD2.DATA_OUT, U2.P0.14
- net MOSI: now also SD1.DATA_IN, U1.P0.13; no longer SD2.DATA_IN, U2.P0.13
- net N$1: now also R11.2; no longer R6.2
- net N$10: now also LED2.A, R7.1; no longer LED4.A, R4.1
- net N$11: now also L1.1, U1.DCC; no longer L2.1, U2.DCC
- net N$12: now also C1.1, L1.2, U1.DEC4; no longer C7.1, L2.2, U2.DEC4
- net N$13: now also C14.2; no longer C16.2
- net N$14: now also DEBUG1.NC/TDI; no longer CORTEX1.NC/TDI
- net N$15: now also C17.2; no longer C18.2
- net N$17: now also CHRG1.PROG, R4.2; no longer CHRG2.PROG, R11.2
- net N$19: now also RTC1.OSCO, XTAL2.1; no longer U4.OSCO, XTAL3.1
- net N$2: now also R14.1; no longer R7.1
- net N$20: now also RTC1.OSCI, XTAL2.2; no longer U4.OSCI, XTAL3.2
- net N$23: now also R12.2, U2.USBDM; no longer R17.2, U5.USBDM
- net N$24: now also R13.2, U2.USBDP; no longer R18.2, U5.USBDP
- net N$25: now also LED3.C, R15.2; no longer LED5.C, R19.2
- net N$26: now also LED4.C, R16.2; no longer LED6.C, R20.2
- net N$3: now also C18.2; no longer C13.2
- net N$4: now also C3.2, U1.P0.00/XL1, XTAL1.1; no longer C8.2, U2.P0.00/XL1, XTAL2.1
- net N$5: now also C18.1; no longer C13.1
- net N$6: now also C5.1, U1.P0.01/XL2, XTAL1.2; no longer C9.1, U2.P0.01/XL2, XTAL2.2
- net N$7: now also C16.2; no longer C15.2
- net N$8: now also C16.1; no longer C15.1
- net N$9: now also LED1.A, R5.1; no longer LED3.A, R3.1
- net P0.09/NFC1: now also U1.P0.09; no longer C11.1, U2.P0.09
- net P0.10/NFC2: now also U1.P0.10; no longer C10.1, U2.P0.10
- net RESET: now also C11.2, D3.A, DEBUG1.!RESET, R10.1, U1.P0.21/RESET; no longer C14.2, CORTEX1.!RESET, D1.A, R5.1, U2.P0.21/RESET
- net RXD.FT: now also R18.1, U2.RXD; no longer R2.1, U5.RXD
- net RXD.NRF: now also R17.2, U1.P0.08; no longer R1.2, U2.P0.08
- net RXLED: now also R15.1, U2.CBUS1; no longer R19.1, U5.CBUS1
- net SCK: now also SD1.SCLK, U1.P0.12; no longer SD2.SCLK, U2.P0.12
- net SCL: now also J2.2, R2.1, RTC1.SCL, U1.P0.26; no longer R9.1, U2.P0.26, U4.SCL
- net SDA: now also J2.1, R1.1, RTC1.SDA, U1.P0.25; no longer R8.1, U2.P0.25, U4.SDA
- net SWCLK: now also DEBUG1.SWDCLK/TCK, U1.SWDCLK; no longer CORTEX1.SWDCLK/TCK, U2.SWDCLK
- net SWDIO: now also DEBUG1.SWDIO/TMS, U1.SWDIO; no longer CORTEX1.SWDIO/TMS, U2.SWDIO
- net SWO: now also DEBUG1.SWO/TDO, U1.P0.18/SWO; no longer CORTEX1.SWO/TDO, U2.P0.18/SWO
- net TXD.FT: now also R17.1, U2.TXD; no longer R1.1, U5.TXD
- net TXD.NRF: now also R18.2, U1.P0.06; no longer R2.2, U2.P0.06
- net TXLED: now also R16.1, U2.CBUS2; no longer R20.1, U5.CBUS2
- net USB+: now also C13.1, R13.1, USB1.D+; no longer C23.1, R18.1, USB2.D+
- net USB-: now also C12.2, R12.1, USB1.D-; no longer C24.2, R17.1, USB2.D-
- net VIN: now also C4.2, C6.2, CHRG1.VIN, D1.C, D2.C, LDO1.EN, LDO1.IN, R3.2; no longer C21.2, C5.2, CHRG2.VIN, D4.C, D5.C, LDO2.EN, LDO2.IN, R12.2
- net VLIPO: now also C10.1, CHRG1.VBAT, D1.A, J1.2, R8.2; no longer C20.1, CHRG2.VBAT, D4.A, J2.2, R13.2
- net V_USB: now also D2.A, U2.VCC, USB1.V+; no longer D5.A, U5.VCC, USB2.V+
Other:
- moved on the sheet: C10, C11, C12, C13, C14, C15, C16, C17, C18, C19, C2, C20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
